Commit message: updated urdf

File: spot_urdf/urdf/spot.urdf (robot description, URDF)
Before this commit: robot spot, 20 links, 19 joints
Joints:
- joint lf_foot_joint: origin xyz=-0.01 0.0 -0.35 rpy=0 0 0 -> xyz=-0.005 0.0 -0.348 rpy=0 0 0
- joint lh_foot_joint: origin xyz=-0.01 0.0 -0.35 rpy=0 0 0 -> xyz=-0.005 0.0 -0.348 rpy=0 0 0
- joint rf_foot_joint: origin xyz=-0.01 0.0 -0.35 rpy=0 0 0 -> xyz=-0.005 0.0 -0.348 rpy=0 0 0
- joint rh_foot_joint: origin xyz=-0.01 0.0 -0.35 rpy=0 0 0 -> xyz=-0.005 0.0 -0.348 rpy=0 0 0
