Commit message: slightly changed foot link position

File: spot_urdf/urdf/spot.urdf.xacro (robot description, xacro)
@@ -60,6 +60,6 @@
     <xacro:property name="foot_mass" value="0.06"/>
     <xacro:property name="foot_radius" value="0.03"/>
-    <xacro:property name="foot_x" value="-0.01"/>
-    <xacro:property name="foot_z" value="-0.35"/>
+    <xacro:property name="foot_x" value="-0.005"/>
+    <xacro:property name="foot_z" value="-0.348"/>
     <xacro:arg name="add_base_joint" default="true"/>
     <xacro:if value="$(arg add_base_joint)">

Commit message: added color to material

File: spot_urdf/urdf/spot.urdf.xacro (robot description, xacro)
@@ -197,5 +197,7 @@
             <sphere radius="${foot_radius-0.01}"/>
         </geometry>
-        <material name="green"/>
+        <material name="green">
+            <color rgba="0.0 0.8 0.0 1.0"/>
+        </material>
     </visual>
     <collision>
@@ -305,5 +307,7 @@
             <sphere radius="${foot_radius-0.01}"/>
         </geometry>
-        <material name="green"/>
+        <material name="green">
+            <color rgba="0.0 0.8 0.0 1.0"/>
+        </material>
     </visual>
     <collision>
@@ -413,5 +417,7 @@
             <sphere radius="${foot_radius-0.01}"/>
         </geometry>
-        <material name="green"/>
+        <material name="green">
+            <color rgba="0.0 0.8 0.0 1.0"/>
+        </material>
     </visual>
     <collision>
@@ -521,5 +527,7 @@
             <sphere radius="${foot_radius-0.01}"/>
         </geometry>
-        <material name="green"/>
+        <material name="green">
+            <color rgba="0.0 0.8 0.0 1.0"/>
+        </material>
     </visual>
     <collision>

Commit message: fixing feet collision && adding cartesio configs

File: spot_urdf/urdf/spot.urdf.xacro (robot description, xacro)
@@ -60,5 +60,5 @@
     <!-- foot -->
     <xacro:property name="foot_mass" value="0.06"/>
-    <xacro:property name="foot_radius" value="0.03"/>
+    <xacro:property name="foot_radius" value="0.02"/>
     <xacro:property name="foot_x" value="-0.005"/>
     <xacro:property name="foot_z" value="-0.348"/>
@@ -187,5 +187,5 @@
     </joint>
     <joint name="lf_foot_joint" type="fixed">
-        <origin xyz="${foot_x} 0.0 ${foot_z}" rpy="0 0 0" />
+        <origin xyz="${foot_x} 0.0 ${foot_z-foot_radius}" rpy="0 0 0" />
         <parent link="lf_lowerleg" />
         <child link="lf_foot" />
@@ -195,5 +195,5 @@
         <origin rpy="0 0 0" xyz="0 0 0"/>
         <geometry>
-            <sphere radius="${foot_radius-0.01}"/>
+            <sphere radius="${0.01}"/>
         </geometry>
         <material name="green">
@@ -201,10 +201,4 @@
         </material>
     </visual>
-    <collision>
-        <origin rpy="0 0 0" xyz="0 0 0"/>
-        <geometry>
-            <sphere radius="${foot_radius}"/>
-        </geometry>
-    </collision>
     <inertial>
         <mass value="${foot_mass}"/>
@@ -297,5 +291,5 @@
     </joint>
     <joint name="rf_foot_joint" type="fixed">
-        <origin xyz="${foot_x} 0.0 ${foot_z}" rpy="0 0 0" />
+        <origin xyz="${foot_x} 0.0 ${foot_z-foot_radius}" rpy="0 0 0" />
         <parent link="rf_lowerleg" />
         <child link="rf_foot" />
@@ -305,5 +299,5 @@
         <origin rpy="0 0 0" xyz="0 0 0"/>
         <geometry>
-            <sphere radius="${foot_radius-0.01}"/>
+            <sphere radius="${0.01}"/>
         </geometry>
         <material name="green">
@@ -311,10 +305,4 @@
         </material>
     </visual>
-    <collision>
-        <origin rpy="0 0 0" xyz="0 0 0"/>
-        <geometry>
-            <sphere radius="${foot_radius}"/>
-        </geometry>
-    </collision>
     <inertial>
         <mass value="${foot_mass}"/>
@@ -407,5 +395,5 @@
     </joint>
     <joint name="lh_foot_joint" type="fixed">
-        <origin xyz="${foot_x} 0.0 ${foot_z}" rpy="0 0 0" />
+        <origin xyz="${foot_x} 0.0 ${foot_z-foot_radius}" rpy="0 0 0" />
         <parent link="lh_lowerleg" />
         <child link="lh_foot" />
@@ -415,5 +403,5 @@
         <origin rpy="0 0 0" xyz="0 0 0"/>
         <geometry>
-            <sphere radius="${foot_radius-0.01}"/>
+            <sphere radius="${0.01}"/>
         </geometry>
         <material name="green">
@@ -421,10 +409,4 @@
         </material>
     </visual>
-    <collision>
-        <origin rpy="0 0 0" xyz="0 0 0"/>
-        <geometry>
-            <sphere radius="${foot_radius}"/>
-        </geometry>
-    </collision>
     <inertial>
         <mass value="${foot_mass}"/>
@@ -517,5 +499,5 @@
     </joint>
     <joint name="rh_foot_joint" type="fixed">
-        <origin xyz="${foot_x} 0.0 ${foot_z}" rpy="0 0 0" />
+        <origin xyz="${foot_x} 0.0 ${foot_z-foot_radius}" rpy="0 0 0" />
         <parent link="rh_lowerleg" />
         <child link="rh_foot" />
@@ -525,5 +507,5 @@
         <origin rpy="0 0 0" xyz="0 0 0"/>
         <geometry>
-            <sphere radius="${foot_radius-0.01}"/>
+            <sphere radius="${0.01}"/>
         </geometry>
         <material name="green">
@@ -531,10 +513,4 @@
         </material>
     </visual>
-    <collision>
-        <origin rpy="0 0 0" xyz="0 0 0"/>
-        <geometry>
-            <sphere radius="${foot_radius}"/>
-        </geometry>
-    </collision>
     <inertial>
         <mass value="${foot_mass}"/>
